File: PCB/WheelSpeedSensorsPCB.kicad_pcb (KiCad board)
At the start: 2 copper layers, 60 x 90 mm, 21 parts, among them J1 RearLeftWheel, J10 FrontRightShock, J11 RearRightShock, J2 FrontRightWheel, J3 RearRightWheel, J4 Conn_01x02_Pin, J5 FrontLeftWheel, J6 RearLeftShock, J7 VehicleBus, J8 Conn_01x02_Pin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

Commit message: Update footprints to better fit standard resistors
Parts:
- R1, R10, R2, R3: footprint Resistor_THT:R_Axial_DIN0204_L3.6mm_D1.6mm_P5.08mm_Horizontal -> Resistor_THT:R_Axial_DIN0204_L3.6mm_D1.6mm_P7.62mm_Horizontal
- moved R10 1.73 mm to (153.2, 117.5)
- moved R3 1.73 mm to (153.2, 122.5)
- moved R1 1.23 mm to (108.7, 122.5)
- moved R2 1.23 mm to (108.7, 117.5)
Routing:
- net Net-(J5-Pin_2): track 75.5 -> 73.7 mm
- net Net-(J3-Pin_2): track 76.2 -> 77.9 mm
- net +5V: track 60.9 -> 59.7 mm
- net Net-(J2-Pin_2): track 87.4 -> 86.9 mm
